File: PowerBoost 500C.brd (EAGLE design)
At the start: 35.6 x 21.6 mm, 42 parts, among them CN1 USBA_FEMALE, Q1 MMUN2133LT1G, U1 TPS61090RSAR, U2 MCP73831T-2ACI/OT, X2 microUSB

Commit message: first commit
Parts:
- removed CN1: USBA_FEMALE, microbuilder:USB_HOST-PTH
- removed JP1: (no value), adafruit:1X06-CLEANBIG
- removed JP2: (no value), microbuilder:1X02_ROUND
- removed R10, R12: 49.9K 1%, microbuilder:0805-NO
- removed R11, R9: 75K 1%, microbuilder:0805-NO
- removed U$25: (no value), microbuilder:SYMBOL_PLUS
- removed U$26: (no value), microbuilder:SYMBOL_MINUS
- removed X1: (no value), microbuilder:TERMBLOCK_1X2-3.5MM
- added J2: (no value), SparkFun-Connectors:JST-2-SMD
- added U$15: MOUNTINGHOLE2.5, microbuilder:MOUNTINGHOLE_2.5_PLATED
Connections:
- removed net D+: CN1.D+, R11.1, R12.1
- removed net D-: CN1.D-, R10.1, R9.1
- net 5.0V: now also J2.1; no longer CN1.VBUS, JP1.6, R11.2, R9.2, X1.2
- net ENABLE: no longer JP1.2
- net GND: now also J2.2; no longer CN1.GND, JP1.3, JP1.5, JP2.2, R10.2, R12.2, X1.1
- net LBO: no longer JP1.4
- net VBAT: no longer JP1.1
- net VDD1: no longer JP2.1
Routing:
- net 5.0V: track 36.2 -> 15.5 mm
- net GND: track 56.4 -> 42.2 mm
- net D+: track 14.0 -> 0.00 mm
- net VDD1: track 19.5 -> 10.00 mm
- net D-: track 4.38 -> 0.00 mm
- net VBAT: track 36.7 -> 32.7 mm
- net ENABLE: track 24.2 -> 21.8 mm
Other:
- board size 35.6 x 21.6 mm -> 38.1 x 21.6 mm
- board text removed: "500C"
- board text removed: "5V"
- board text removed: "Boost"
- board text removed: "LB"
- board text removed: "Power"
- board text removed: "adafruit"
